Commit message: Improve docker

File: src/mk_mini_simulator/urdf/mk_mini.urdf.xacro (robot description, xacro)
@@ -5,9 +5,27 @@
     <xacro:property name="chassis_width" value="0.60"/>
     <xacro:property name="chassis_height" value="0.31"/>
+    <xacro:property name="chassis_mass" value="40.0"/>
     <xacro:property name="ground_clearance" value="0.111"/>
     <xacro:property name="wheel_radius" value="0.12"/>
     <xacro:property name="wheel_width" value="0.08"/>
+    <xacro:property name="wheel_mass" value="2.5"/>
     <xacro:property name="wheelbase" value="0.60"/>
     <xacro:property name="track_width" value="0.517"/>
+    <xacro:macro name="box_inertia" params="m x y z">
+        <inertial>
+            <mass value="${m}"/>
+            <inertia ixx="${(m/12) * (y*y + z*z)}" ixy="0.0" ixz="0.0"
+                     iyy="${(m/12) * (x*x + z*z)}" iyz="0.0"
+                     izz="${(m/12) * (x*x + y*y)}"/>
+        </inertial>
+    </xacro:macro>
+    <xacro:macro name="cylinder_inertia" params="m r h">
+        <inertial>
+            <mass value="${m}"/>
+            <inertia ixx="${(m/12) * (3*r*r + h*h)}" ixy="0.0" ixz="0.0"
+                     iyy="${(m/12) * (3*r*r + h*h)}" iyz="0.0"
+                     izz="${(m/2) * (r*r)}"/>
+        </inertial>
+    </xacro:macro>
     <link name="base_footprint"/>
     <link name="base_link">
@@ -16,8 +34,12 @@
                 <box size="${chassis_length} ${chassis_width} ${chassis_height}"/>
             </geometry>
-            <material name="translucent_white">
-                <color rgba="0.9 0.9 0.9 0.4"/>
-            </material>
+            <material name="translucent_white"><color rgba="0.9 0.9 0.9 0.4"/></material>
         </visual>
+        <collision>
+            <geometry>
+                <box size="${chassis_length} ${chassis_width} ${chassis_height}"/>
+            </geometry>
+        </collision>
+        <xacro:box_inertia m="${chassis_mass}" x="${chassis_length}" y="${chassis_width}" z="${chassis_height}"/>
     </link>
     <joint name="base_joint" type="fixed">
@@ -29,11 +51,11 @@
         <link name="${prefix}_rear_wheel">
             <visual>
-                <geometry>
-                    <cylinder radius="${wheel_radius}" length="${wheel_width}"/>
-                </geometry>
-                <material name="black">
-                    <color rgba="0.1 0.1 0.1 1.0"/>
-                </material>
+                <geometry><cylinder radius="${wheel_radius}" length="${wheel_width}"/></geometry>
+                <material name="black"><color rgba="0.1 0.1 0.1 1.0"/></material>
             </visual>
+            <collision>
+                <geometry><cylinder radius="${wheel_radius}" length="${wheel_width}"/></geometry>
+            </collision>
+            <xacro:cylinder_inertia m="${wheel_mass}" r="${wheel_radius}" h="${wheel_width}"/>
         </link>
         <joint name="${prefix}_rear_wheel_joint" type="continuous">
@@ -43,15 +65,17 @@
             <axis xyz="0 0 -1"/>
         </joint>
+        <gazebo reference="${prefix}_rear_wheel">
+            <mu1>1.0</mu1>
+            <mu2>1.0</mu2>
+            <material>Gazebo/DarkGrey</material>
+        </gazebo>
     </xacro:macro>
     <xacro:macro name="front_wheel_steering" params="prefix y_reflect">
         <link name="${prefix}_steering_knuckle">
             <visual>
-                <geometry>
-                    <box size="0.06 0.06 0.06"/>
-                </geometry>
-                <material name="grey">
-                    <color rgba="0.5 0.5 0.5 1.0"/>
-                </material>
+                <geometry><box size="0.06 0.06 0.06"/></geometry>
+                <material name="grey"><color rgba="0.5 0.5 0.5 1.0"/></material>
             </visual>
+            <xacro:box_inertia m="0.5" x="0.06" y="0.06" z="0.06"/>
         </link>
         <joint name="${prefix}_steering_joint" type="revolute">
@@ -60,15 +84,15 @@
             <origin xyz="${wheelbase/2.0} ${y_reflect * track_width/2.0} ${-chassis_height/2.0 + (wheel_radius - ground_clearance)}" rpy="0 0 0"/>
             <axis xyz="0 0 1"/>
-            <limit lower="-0.6" upper="0.6" effort="10.0" velocity="1.0"/>
+            <limit lower="-0.6" upper="0.6" effort="100.0" velocity="2.0"/>
         </joint>
         <link name="${prefix}_front_wheel">
             <visual>
-                <geometry>
-                    <cylinder radius="${wheel_radius}" length="${wheel_width}"/>
-                </geometry>
-                <material name="black_wheels">
-                    <color rgba="0.1 0.1 0.1 1.0"/>
-                </material>
+                <geometry><cylinder radius="${wheel_radius}" length="${wheel_width}"/></geometry>
+                <material name="black"><color rgba="0.1 0.1 0.1 1.0"/></material>
             </visual>
+            <collision>
+                <geometry><cylinder radius="${wheel_radius}" length="${wheel_width}"/></geometry>
+            </collision>
+            <xacro:cylinder_inertia m="${wheel_mass}" r="${wheel_radius}" h="${wheel_width}"/>
         </link>
         <joint name="${prefix}_front_wheel_joint" type="continuous">
@@ -78,4 +102,9 @@
             <axis xyz="0 0 -1"/>
         </joint>
+        <gazebo reference="${prefix}_front_wheel">
+            <mu1>0.8</mu1>
+            <mu2>0.8</mu2>
+            <material>Gazebo/DarkGrey</material>
+        </gazebo>
     </xacro:macro>
     <xacro:rear_wheel prefix="left" y_reflect="1"/>
@@ -83,3 +112,29 @@
     <xacro:front_wheel_steering prefix="left" y_reflect="1"/>
     <xacro:front_wheel_steering prefix="right" y_reflect="-1"/>
+    <gazebo>
+        <plugin name="gazebo_ros_ackermann_drive" filename="libgazebo_ros_ackermann_drive.so">
+            <update_rate>50.0</update_rate>
+            <front_left_joint>left_steering_joint</front_left_joint>
+            <front_right_joint>right_steering_joint</front_right_joint>
+            <rear_left_joint>left_rear_wheel_joint</rear_left_joint>
+            <rear_right_joint>right_rear_wheel_joint</rear_right_joint>
+            <wheel_separation>${track_width}</wheel_separation>
+            <wheel_diameter>${wheel_radius * 2.0}</wheel_diameter>
+            <wheelbase>${wheelbase}</wheelbase>
+            <max_steer>0.6</max_steer>
+            <max_speed>3.0</max_speed>
+            <max_steering_angle>0.6</max_steering_angle>
+            <max_steering_rate>1.0</max_steering_rate>
+            <ros>
+                <remapping>cmd_vel:=cmd_vel</remapping>
+                <remapping>odom:=odom</remapping>
+            </ros>
+            <publish_odom>true</publish_odom>
+            <publish_odom_tf>true</publish_odom_tf>
+            <publish_wheel_tf>true</publish_wheel_tf>
+            <publish_distance_aware_steering>true</publish_distance_aware_steering>
+            <odometry_frame>odom</odometry_frame>
+            <robot_base_frame>base_footprint</robot_base_frame>
+        </plugin>
+    </gazebo>
 </robot>

Commit message: Improve simulator

File: src/mk_mini_simulator/urdf/mk_mini.urdf.xacro (robot description, xacro)
@@ -27,4 +27,54 @@
                      izz="${(m/2) * (r*r)}"/>
         </inertial>
+    </xacro:macro>
+    <xacro:macro name="ultrasonic_sensor" params="prefix x y z yaw">
+        <link name="sonar_${prefix}">
+            <visual>
+                <geometry><box size="0.02 0.04 0.02"/></geometry>
+                <material name="grey"><color rgba="0.5 0.5 0.5 1.0"/></material>
+            </visual>
+            <xacro:box_inertia m="0.05" x="0.02" y="0.04" z="0.02"/>
+        </link>
+        <joint name="sonar_${prefix}_joint" type="fixed">
+            <parent link="base_link"/>
+            <child link="sonar_${prefix}"/>
+            <origin xyz="${x} ${y} ${z}" rpy="0 0 ${yaw}"/>
+        </joint>
+        <gazebo reference="sonar_${prefix}">
+            <sensor type="ray" name="sonar_${prefix}_sensor">
+                <always_on>true</always_on>
+                <update_rate>20.0</update_rate> <visualize>true</visualize> <ray>
+                    <scan>
+                        <horizontal>
+                          <samples>5</samples>
+			  <resolution>1</resolution>
+                          <min_angle>-0.13</min_angle>
+			  <max_angle>0.13</max_angle>
+                        </horizontal>
+			<!--
+                        <vertical>
+                            <samples>5</samples>
+                            <resolution>1</resolution>
+                            <min_angle>-0.05</min_angle>
+                            <max_angle>0.05</max_angle>
+                        </vertical>
+			-->
+                    </scan>
+                    <range>
+                      <min>0.05</min>
+		      <max>3.00</max>
+		      <resolution>0.001</resolution>
+		    </range>
+                </ray>
+                <plugin name="gazebo_ros_sonar_${prefix}" filename="libgazebo_ros_ray_sensor.so">
+                    <ros>
+                        <remapping>~/out:=/simulation/sonar_${prefix}</remapping>
+                    </ros>
+                    <output_type>sensor_msgs/Range</output_type>
+                    <frame_name>sonar_${prefix}</frame_name>
+                    <radiation_type>ultrasound</radiation_type>
+		</plugin>
+            </sensor>
+        </gazebo>
     </xacro:macro>
     <link name="base_footprint"/>
@@ -112,11 +162,35 @@
     <xacro:front_wheel_steering prefix="left" y_reflect="1"/>
     <xacro:front_wheel_steering prefix="right" y_reflect="-1"/>
+    <xacro:ultrasonic_sensor prefix="front_center" x="0.42" y="0.0" z="0.0" yaw="0.0"/>
+    <xacro:ultrasonic_sensor prefix="front_left"   x="0.40" y="0.25" z="0.0" yaw="0.4"/>
+    <xacro:ultrasonic_sensor prefix="front_right"  x="0.40" y="-0.25" z="0.0" yaw="-0.4"/>
+    <xacro:ultrasonic_sensor prefix="rear_center"  x="-0.42" y="0.0" z="0.0" yaw="${PI}"/>
+    <xacro:ultrasonic_sensor prefix="rear_left"    x="-0.40" y="0.25" z="0.0" yaw="${PI - 0.4}"/>
+    <xacro:ultrasonic_sensor prefix="rear_right"   x="-0.40" y="-0.25" z="0.0" yaw="${PI + 0.4}"/>
+    <xacro:ultrasonic_sensor prefix="side_left"    x="0.0" y="0.30" z="0.0" yaw="${PI/2}"/>
+    <xacro:ultrasonic_sensor prefix="side_right"   x="0.0" y="-0.30" z="0.0" yaw="${-PI/2}"/>
+    <link name="steering_wheel_link">
+        <visual>
+            <geometry><cylinder radius="0.01" length="0.01"/></geometry>
+            <material name="translucent_white"><color rgba="0 0 0 0"/></material>
+        </visual>
+        <xacro:cylinder_inertia m="0.01" r="0.01" h="0.01"/>
+    </link>
+    <joint name="steering_wheel_joint" type="continuous">
+        <parent link="base_link"/>
+        <child link="steering_wheel_link"/>
+        <origin xyz="0 0 0" rpy="0 0 0"/>
+        <axis xyz="0 0 1"/>
+    </joint>
     <gazebo>
         <plugin name="gazebo_ros_ackermann_drive" filename="libgazebo_ros_ackermann_drive.so">
             <update_rate>50.0</update_rate>
-            <front_left_joint>left_steering_joint</front_left_joint>
-            <front_right_joint>right_steering_joint</front_right_joint>
+            <front_left_joint>left_front_wheel_joint</front_left_joint>
+            <front_right_joint>right_front_wheel_joint</front_right_joint>
             <rear_left_joint>left_rear_wheel_joint</rear_left_joint>
             <rear_right_joint>right_rear_wheel_joint</rear_right_joint>
+            <left_steering_joint>left_steering_joint</left_steering_joint>
+            <right_steering_joint>right_steering_joint</right_steering_joint>
+            <steering_wheel_joint>steering_wheel_joint</steering_wheel_joint>
             <wheel_separation>${track_width}</wheel_separation>
             <wheel_diameter>${wheel_radius * 2.0}</wheel_diameter>
